File: F405_pill_V1.1/F405_pill.kicad_pcb (KiCad board)
At the start: 4 copper layers, 70.5 x 26.6 mm, 64 parts, among them J1 Conn_01x04_Male, J2 Conn_01x04_Male, J3 Conn_01x04_Male, J4 TYPE-C-31-M-12, J5 Conn_01x02, U1 STM32F405VGTx, U2 TJA1050T/CM,118, U3 LM1117-3.3, U4 STM32F405_pill, U5 HT7550, U6 E73-2G4M08S1C, U8 LSM6DS3, Y1 8MHz

Commit message: updated for prodaction
Parts:
- removed U3: LM1117-3.3, Package_TO_SOT_SMD:SOT-223-3_TabPin2
- added U7: AMS1117-3.3, Package_TO_SOT_SMD:SOT-223-3_TabPin2, F.Cu at (130.2, 87.5)
Routing:
- net +3V3: vias 13 -> 12
