File: F405_pill_V1.1/nrf.kicad_sch (KiCad schematic)
At the start: 4 parts, among them U6 E73-2G4M08S1C

Commit message: Schematic is finished
Parts:
- added J3: Conn_01x04_Male, Connector_PinHeader_2.54mm:PinHeader_1x04_P2.54mm_Vertical, symbol Connector:Conn_01x04_Male
- U6: footprint E73-2G4M08S1C:E73-2G4M08S1C -> CCC_ESC_Custom_parts:E73-2G4M08S1C
Connections:
- net +3V3: now also J3.4 (Pin_4)
- net GND: now also J3.1 (Pin_1)
- net at U6.37 (SWDIO): now also J3.3 (Pin_3)
- net at U6.39 (SWDCLK): now also J3.2 (Pin_2)
Other:
- note added: "ST-LINK"
